File: keyboard.kicad_pcb (KiCad board)
At the start: 2 copper layers, 228 x 75.8 mm, 186 parts, among them IC1 ATMEGA32U4, J1 MINI, P1 MISO, P10 GPIO3, P16 Vcc, P17 GND, P18 Row1, P19 Row2, P2 Vcc, P20 Row3, P200 GND, P201 GND, P202 GND, P203 GND, P204 GND, P205 GND, P21 Row4, P23 Col1, P24 Col2, P25 Col3, P26 Col4, P27 Col5, P28 Col6, P29 Col7, P3 SCK, P30 Col8, P31 Col9, P32 Col10, P33 Col11, P34 Col12, P37 Vcc, P38 GPIO0, P39 GPIO1, P4 MOSI, P40 GPIO2, P41 GPIO3, P42 GND, P5 RES, P6 GND, P7 GPIO0, P8 GPIO1, P9 GPIO2, X1 ASX3F

Commit message: v0.4
Parts:
- added DB481: LED, MX_LED, B.Cu at (257.1, 111.9)
- added DB531: LED, MX_LED, B.Cu at (278.7, 111.9)
- added H5: HOLE, PKRHSL, F.Cu at (288.5, 121.1)
- added S481: MX1A, CHERRY_PCB_100H_Plated, F.Cu at (257.1, 111.9)
- added S531: MX1A, CHERRY_PCB_125H_Visible, F.Cu at (278.7, 111.9)
- H1: footprint PKRHC -> PKRH
- S29: footprint CHERRY_PCB_625H-flip -> CHERRY_PCB_625H-FlipPlated
- moved H4 23.1 mm to (262.2, 92.9)
- moved H1 19.3 mm to (105.0, 84.2)
- moved D53 4.22 mm to (280.7, 120.0), turned to 180 degrees
- moved RW2 2.29 mm to (103.7, 93.9)
Connections:
- D48 pad 1: /Matrix/col10 -> N-0000093
- D48 pad 2: N-0000095 (its old number) -> /Matrix/col10
- D53 pad 1: /Matrix/col11 -> N-0000094
- D53 pad 2: N-00000102 (its old number) -> /Matrix/col11
- S48 pad 2: N-0000095 (its old number) -> N-0000093
- S53 pad 2: N-00000102 (its old number) -> N-0000094
Routing:
- net GND: track 628.1 -> 733.1 mm, vias 6 -> 13
- net VCC: track 472.7 -> 421.5 mm, vias 7 -> 9
- net /Matrix/row1: track 335.1 -> 288.7 mm, vias 1 -> 2
- net /Matrix/row2: track 302.8 -> 258.3 mm
- net /GPIO1: track 271.2 -> 239.8 mm, vias 5 -> 3
- net /Matrix/col9: track 106.8 -> 138.1 mm, vias 2 -> 4
- net /Matrix/row3: track 236.1 -> 263.4 mm, vias 2 -> 1
- net /Matrix/col1: track 200.6 -> 222.6 mm
- net /Matrix/CAPS_LED: track 206.0 -> 186.3 mm
- net /Matrix/col7: track 82.0 -> 101.4 mm
- net /Leds/lrow1: track 223.8 -> 242.5 mm
- net N-0000016: track 162.9 -> 181.2 mm
- net /~RES~: track 162.1 -> 179.2 mm, vias 3 -> 4
- net N-0000018: track 153.6 -> 169.2 mm
- net /Matrix/col4: track 131.2 -> 117.2 mm
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
Commit message: v0.5
Parts:
- removed P10: GPIO3, pad
- removed P16: Vcc, pad
- removed P17: GND, pad
- removed P7: GPIO0, pad
- removed P8: GPIO1, pad
- removed P9: GPIO2, pad
Routing:
- net GND: track 733.1 -> 949.9 mm, vias 13 -> 25
- net /GPIO3: track 175.6 -> 95.6 mm, vias 1 -> 0
- net /GPIO2: track 166.7 -> 96.9 mm, vias 2 -> 1
- net /Matrix/col11: track 140.5 -> 193.8 mm, vias 2 -> 0
- net VCC: track 421.5 -> 394.4 mm, vias 9 -> 8
- net /Matrix/col1: track 222.6 -> 197.0 mm
- net /Matrix/row3: track 263.4 -> 241.3 mm, vias 1 -> 0
- net /Matrix/CAPS_LED: track 186.3 -> 164.5 mm, vias 2 -> 1
- net /Matrix/col7: track 101.4 -> 84.9 mm
- net /GPIO0: track 259.7 -> 244.5 mm, vias 1 -> 0
- net N-0000023: track 181.2 -> 166.1 mm
- net /Matrix/col9: track 138.1 -> 123.1 mm, vias 4 -> 0
- net /~RES~: track 179.2 -> 166.0 mm, vias 4 -> 2
- net /Leds/lrow1: track 242.5 -> 229.3 mm
- net /Leds/lcol6: track 116.9 -> 104.9 mm, vias 1 -> 0
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Other:
- board text removed: "+"
- board text removed: "-"
- board text removed: "0"
- board text removed: "1"
- board text removed: "2"
- board text removed: "3"

Commit message: v0.6
Parts:
- added P10: ROW4, Pad_50mil, B.Cu at (288.3, 88.9)
- added P11: ROW5, Pad_50mil, B.Cu at (288.3, 90.2)
- added P43: GPIO3, Pad_50mil, B.Cu at (288.3, 100.3)
- added P44: GPIO6, Pad_50mil, B.Cu at (288.3, 101.6)
- added P45: GND, Pad_50mil, B.Cu at (288.3, 102.9)
- added P7: ROW1, Pad_50mil, B.Cu at (288.3, 85.1)
- added P8: ROW2, Pad_50mil, B.Cu at (288.3, 86.4)
- added P9: ROW3, Pad_50mil, B.Cu at (288.3, 87.6)
- H1, H3, H4: footprint PKRH -> Mechanical_Slotted_Hole
- H2, H5: footprint PKRHSL -> Mechanical_Slot
- P18: value Row1 -> LR1; footprint pad -> Pad_50mil; moved to B.Cu
- P19: value Row2 -> LR2; footprint pad -> Pad_50mil; moved to B.Cu
- P20: value Row3 -> LR3; footprint pad -> Pad_50mil; moved to B.Cu
- P200, P201, P202, P203, P204, P205: footprint Pad-Gnd -> Pad_Gnd
- P21: value Row4 -> LR4; footprint pad -> Pad_50mil; moved to B.Cu
- P23: value Col1 -> LC1; footprint pad -> Pad_50mil; moved to B.Cu
- P24: value Col2 -> LC2; footprint pad -> Pad_50mil; moved to B.Cu
- P25: value Col3 -> LC3; footprint pad -> Pad_50mil; moved to B.Cu
- P26: value Col4 -> LC4; footprint pad -> Pad_50mil; moved to B.Cu
- P27: value Col5 -> LC5; footprint pad -> Pad_50mil; moved to B.Cu
- P28: value Col6 -> LC6; footprint pad -> Pad_50mil; moved to B.Cu
- P29: value Col7 -> LC7; footprint pad -> Pad_50mil; moved to B.Cu
- P30: value Col8 -> LC8; footprint pad -> Pad_50mil; moved to B.Cu
- P31: value Col9 -> LC9; footprint pad -> Pad_50mil; moved to B.Cu
- P32: value Col10 -> LC10; footprint pad -> Pad_50mil; moved to B.Cu
- P33: value Col11 -> LC11; footprint pad -> Pad_50mil; moved to B.Cu
- P34: value Col12 -> LC12; footprint pad -> Pad_50mil; moved to B.Cu
- P37, P38, P39, P40, P41: footprint pad -> Pad_50mil; moved to B.Cu
- P42: value GND -> GPIO2; footprint pad -> Pad_50mil; moved to B.Cu
- moved P42 76.7 mm to (288.3, 99.1), turned to 270 degrees
- moved P41 61.0 mm to (288.3, 97.8), turned to 270 degrees
- moved P38 60.5 mm to (288.3, 94.0), turned to 270 degrees
- moved P39 59.0 mm to (288.3, 95.2), turned to 270 degrees
- moved P40 58.5 mm to (288.3, 96.5), turned to 270 degrees
- moved P37 56.6 mm to (288.3, 92.7), turned to 270 degrees
- moved P31 20.5 mm to (214.4, 68.6), turned to 270 degrees
- moved P27 20.0 mm to (195.6, 68.6), turned to 270 degrees
- moved P32 19.4 mm to (214.4, 69.8), turned to 270 degrees
- moved P18 10.2 mm to (157.5, 68.6), turned to 270 degrees
- moved P23 10.2 mm to (176.3, 68.6), turned to 270 degrees
- moved P30 6.36 mm to (195.6, 72.4), turned to 270 degrees
- moved P25 5.08 mm to (176.3, 71.1), turned to 270 degrees
- moved P21 3.82 mm to (157.5, 72.4), turned to 270 degrees
- moved P26 3.81 mm to (176.3, 72.4), turned to 270 degrees
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Connections:
- net /MISO renamed /GPIO6
- IC1 pad 22: (no net) -> /GPIO5
- IC1 pad 26: (no net) -> /GPIO4
- IC1 pad 8: (no net) -> /row5
- P42 pad 1: GND -> /GPIO4
Routing:
- net GND: track 949.9 -> 670.9 mm, vias 25 -> 5
- net /GPIO5: track 0.00 -> 117.1 mm, vias 0 -> 2
- net /GPIO4: track 0.00 -> 108.5 mm, vias 0 -> 2
- net /row5: track 0.00 -> 97.3 mm, vias 0 -> 1
- net /GPIO6: track 66.6 -> 161.8 mm
- net /Matrix/row4: track 212.4 -> 265.2 mm, vias 1 -> 2
- net /Matrix/row3: track 241.3 -> 285.4 mm, vias 0 -> 2
- net /GPIO0: track 244.5 -> 281.8 mm, vias 0 -> 1
- net VCC: track 394.4 -> 422.8 mm
- net /Leds/lcol3: track 98.7 -> 124.3 mm, vias 0 -> 1
- net /Leds/lcol10: track 132.4 -> 108.0 mm, vias 0 -> 1
- net /Matrix/col10: track 150.5 -> 174.4 mm, vias 0 -> 2
- net /Leds/lcol9: track 120.4 -> 98.0 mm
- net /GPIO3: track 95.6 -> 116.3 mm, vias 0 -> 1
- net /GPIO2: track 96.9 -> 117.2 mm
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Other:
- board text added: "Rev 0.6"

Commit message: v0.7
Parts:
- removed P11: ROW5, Pad_50mil
- added P46: GND, Pad_50mil, B.Cu at (288.3, 102.9)
- J1: footprint 67503 -> USB_MINI-B_MOLEX_67503-1020
- P42: value GPIO2 -> GPIO4
- P43: value GPIO3 -> GPIO5
- P45: value GND -> GPIO7
- moved P38 1.27 mm to (288.3, 92.7)
- moved P41 1.27 mm to (288.3, 96.5)
- moved P45 1.27 mm to (288.3, 101.6)
- moved P37 1.27 mm to (288.3, 91.4)
- moved P39 1.27 mm to (288.3, 94.0)
- moved P40 1.27 mm to (288.3, 95.2)
- moved P42 1.27 mm to (288.3, 97.8)
- moved P43 1.27 mm to (288.3, 99.1)
- moved P44 1.27 mm to (288.3, 100.3)
Connections:
- IC1 pad 8: /row5 -> /GPIO7
- P45 pad 1: GND -> /GPIO7
Routing:
- net /GPIO7: track 0.00 -> 110.7 mm, vias 0 -> 1
- net /row5: track 97.3 -> 0.00 mm, vias 1 -> 0
- net VCC: track 422.8 -> 505.7 mm, vias 8 -> 1
- net GND: track 670.9 -> 596.5 mm, vias 5 -> 12
- net /Matrix/col11: track 186.4 -> 144.2 mm, vias 3 -> 2
- net /~RES~: track 177.3 -> 157.0 mm, vias 3 -> 1
- net /GPIO5: track 117.1 -> 103.4 mm, vias 2 -> 1
- net /GPIO0: track 281.8 -> 294.4 mm, vias 1 -> 0
- net /Matrix/col10: track 174.4 -> 162.7 mm, vias 2 -> 0
- net /Matrix/row3: track 285.4 -> 274.8 mm
- net /GPIO6: track 161.8 -> 172.2 mm
- net /Leds/lcol11: track 112.2 -> 102.0 mm
- net /Matrix/row4: track 265.2 -> 274.7 mm, vias 2 -> 1
- net /Leds/lcol10: track 108.0 -> 116.5 mm, vias 1 -> 0
- net /Matrix/col4: track 117.9 -> 109.5 mm, vias 2 -> 0
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Other:
- board text added: "Interconnect Pads Pinout on Reverse"
- board text added: "LEDs"
- board text added: "Note LED Rotation for Alternate S531 & S481 Switch Placements"
- board text added: "Rev 0.7"
- board text added: "S01"
- board text added: "S01LED"
- board text added: "S02"
- board text added: "S02 LED"
- board text added: "S03"
- board text added: "S04"
- board text added: "S06"
- board text added: "S07"
- board text added: "S07 'A' LED"
- board text added: "S08"
- board text added: "S09"
- board text added: "S11"
- board text added: "S11 'W' LED"
- board text added: "S12"
- board text added: "S12 'S' LED"
- board text added: "S13"
- board text added: "S14"
- board text added: "S16"
- board text added: "S16 'D' LED"
- board text added: "S17"
- board text added: "S18"
- board text added: "S21"
- board text added: "S22"
- board text added: "S23"
- board text added: "S26"
- board text added: "S27"
- board text added: "S28"
- board text added: "S29"
- board text added: "S31"
- board text added: "S32"
- board text added: "S33"
- board text added: "S36"
- board text added: "S37"
- board text added: "S38"
- board text added: "S41"
- board text added: "S42"
- board text added: "S43"
- board text added: "S44"
- board text added: "S46"
- board text added: "S47"
- board text added: "S48"
- board text added: "S481"
- board text added: "S49"
- board text added: "S51"
- board text added: "S52"
- board text added: "S53"
- board text added: "S531"
- board text added: "S56"
- board text added: "Special thanks to komar007, bpiphany, Dox, jdcarpe and Regack"
- board text added: "orD481"
- board text removed: "CAPS"
- board text removed: "ESC"
- board text removed: "GPIO"
- board text removed: "Rev 0.6"
- board text removed: "Special thanks to komar007, bpiphany, Dox and Regack"

Commit message: v0.10
Parts:
- removed P204, P205: GND, Pad_Gnd
- added P35: LGND, Pad, B.Cu at (195.9, 80.2)
- added P36: LVcc, Pad, B.Cu at (214.9, 80.2)
- added P47: GND, Pad_50mil, B.Cu at (288.3, 102.9)
- D01, D02, D03, D04, D06, D07, D08, D09, D11, D12, D13, D14, D16, D17, D18, D21, D22, D23, D26, D27, D28, D29, D31, D32, D33, D36, D37, D38, D41, D42, D43, D44, D46, D47, D48, D49, D51, D52, D53, D56: footprint SM0805D -> SOD-123
- H1, H3, H4: footprint Mechanical_Slotted_Hole -> Mechanical_Hole
- H2, H5: footprint Mechanical_Slot -> Mechanical_Hole
- P18, P19, P20, P21, P23, P24, P25, P26, P27, P28, P29, P30, P31, P32, P33, P34: footprint Pad_50mil -> Pad
- P42: value GPIO4 -> GPIO4(SS)
- P43: value GPIO5 -> GPIO5(SCK)
- P44: value GPIO6 -> GPIO6(MOSI)
- P45: value GPIO7 -> GPIO7(SCL)
- P46: value GND -> GPIO8(SDA)
- S29: footprint CHERRY_PCB_625H-FlipPlated -> CHERRY_PCB_625H_Rev
- moved D04 8.52 mm to (78.4, 125.9), turned to 90 degrees
- moved D09 8.52 mm to (100.0, 125.9), turned to 90 degrees
- moved D14 8.52 mm to (119.1, 125.9), turned to 90 degrees
- moved D44 8.25 mm to (260.0, 125.9), turned to 90 degrees
- moved D49 8.25 mm to (283.5, 125.9), turned to 90 degrees
- moved D29 8.25 mm to (188.3, 125.9), turned to 90 degrees
- moved D48 7.24 mm to (261.9, 118.9), turned to 270 degrees
- moved D08 6.75 mm to (107.6, 118.9), turned to 270 degrees
- moved D13 6.75 mm to (126.7, 118.9), turned to 270 degrees
- moved D18 6.75 mm to (145.7, 118.9), turned to 270 degrees
- moved D23 6.75 mm to (164.8, 118.9), turned to 270 degrees
- moved D33 6.75 mm to (202.9, 118.9), turned to 270 degrees
- moved D38 6.75 mm to (221.9, 118.9), turned to 270 degrees
- moved D43 6.75 mm to (241.0, 118.9), turned to 270 degrees
- moved D37 6.75 mm to (213.0, 99.9), turned to 270 degrees
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Connections:
- D56 pad 1: /Matrix/col12 -> /Matrix/col11
- IC1 pad 1: /Matrix/col3 -> /GPIO2
- IC1 pad 10: /Matrix/CAPS_LED -> /GPIO6
- IC1 pad 11: /GPIO6 -> /Matrix/col7
- IC1 pad 12: /Matrix/col9 -> /Matrix/col11
- IC1 pad 18: /Matrix/row1 -> /GPIO7
- IC1 pad 19: /Matrix/row2 -> /GPIO8
- IC1 pad 20: /Matrix/row3 -> /Matrix/row1
- IC1 pad 21: /Matrix/row4 -> /Matrix/row2
- IC1 pad 22: /GPIO5 -> /Matrix/row4
- IC1 pad 25: /Matrix/col7 -> /Matrix/row3
- IC1 pad 26: /GPIO4 -> /GPIO0
- IC1 pad 27: /Matrix/col12 -> /GPIO1
- IC1 pad 28: /Matrix/col11 -> /Matrix/col8
- IC1 pad 29: /Matrix/col10 -> /Matrix/col9
- IC1 pad 30: /Matrix/col6 -> /Matrix/col10
- IC1 pad 31: /Matrix/col5 -> /Matrix/CAPS_LED
- IC1 pad 32: /Matrix/col4 -> /GPIO3
- IC1 pad 36: /GPIO0 -> /Matrix/col6
- IC1 pad 37: /GPIO1 -> /Matrix/col5
- IC1 pad 38: /GPIO2 -> /Matrix/col4
- IC1 pad 39: /GPIO3 -> /Matrix/col3
- IC1 pad 8: /GPIO7 -> /GPIO4
- IC1 pad 9: /Matrix/col8 -> /GPIO5
- P1 pad 1: /GPIO6 -> /Matrix/col7
- P3 pad 1: /Matrix/col8 -> /GPIO5
- P4 pad 1: /Matrix/CAPS_LED -> /GPIO6
- P46 pad 1: GND -> /GPIO8
- S56 pad 1: /Matrix/row1 -> /Matrix/row4
Routing:
- net GND: track 596.5 -> 789.6 mm, vias 12 -> 26
- net /Matrix/col12: track 126.4 -> 0.00 mm, vias 2 -> 0
- net /GPIO8: track 0.00 -> 100.6 mm, vias 0 -> 3
- net /GPIO5: track 103.4 -> 169.9 mm, vias 1 -> 4
- net /Matrix/col9: track 108.5 -> 162.8 mm
- net /Matrix/col8: track 133.7 -> 92.1 mm, vias 3 -> 2
- net /Matrix/col7: track 85.7 -> 121.3 mm, vias 2 -> 3
- net VCC: track 505.7 -> 472.4 mm, vias 1 -> 2
- net /Leds/lrow3: track 305.3 -> 275.9 mm, vias 0 -> 1
- net /GPIO1: track 262.7 -> 291.2 mm, vias 1 -> 2
- net /Matrix/col4: track 109.5 -> 131.7 mm
- net /Leds/lcol8: track 53.6 -> 71.8 mm
- net /Matrix/CAPS_LED: track 169.2 -> 152.8 mm, vias 2 -> 1
- net /Leds/lcol6: track 113.6 -> 97.6 mm
- net /GPIO0: track 294.4 -> 279.0 mm, vias 0 -> 1
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Other:
- outline, holes or cut-outs redrawn
- net class Default: clearance 0.2032 -> 0.2; trace_width 0.4064 -> 0.2; via_dia 1 -> 0.8
- net class POWER: clearance 0.2032 -> 0.2; trace_width 0.508 -> 0.4
- rule trace_clearance: 0.2032 -> 0.2
- rule trace_min: 0.2032 -> 0.2
- rule via_min_size: 1 -> 0.8
- board text added: "Rev 0.10"
- board text added: "S03 LED"
- board text added: "orD531"
- board text removed: "Rev 0.7"
- board text removed: "S02 LED"
