File: keyboard.sch (KiCad schematic (older format))
At the start: 66 parts, among them IC1 ATMEGA32U4, J1 MINI, P1 MISO, P10 GPIO3, P16 Vcc, P17 GND, P18 Row1, P19 Row2, P2 Vcc, P20 Row3, P200 GND, P201 GND, P202 GND, P203 GND, P204 GND, P205 GND, P21 Row4, P23 Col1, P24 Col2, P25 Col3, P26 Col4, P27 Col5, P28 Col6, P29 Col7, P3 SCK, P30 Col8, P31 Col9, P32 Col10, P33 Col11, P34 Col12, P37 Vcc, P38 GPIO0, P39 GPIO1, P4 MOSI, P40 GPIO2, P41 GPIO3, P42 GND, P5 RES, P6 GND, P7 GPIO0, P8 GPIO1, P9 GPIO2, X1 ASX3F

Commit message: v0.5
Parts:
- removed P10: GPIO3, symbol CONN_1
- removed P16: Vcc, symbol CONN_1
- removed P17: GND, symbol CONN_1
- removed P7: GPIO0, symbol CONN_1
- removed P8: GPIO1, symbol CONN_1
- removed P9: GPIO2, symbol CONN_1
Other:
- note removed: "Universal expansion\nconnector (bottom)"
Changed lines of the file:
@@
-EESchema Schematic File Version 2  date 9/20/2013 9:26:52 AM
+EESchema Schematic File Version 2  date 9/20/2013 1:35:54 PM
 LIBS:power
 LIBS:mx1a-simple
@@
 GPIO3
 $Comp
-L CONN_1 P7
-U 1 1 5136239B
-P 9800 6150
-F 0 "P7" H 9880 6150 40  0000 L CNN
-F 1 "GPIO0" H 9800 6205 30  0001 C CNN
-F 2 "" H 9800 6150 60  0001 C CNN
-F 3 "" H 9800 6150 60  0001 C CNN
-	1    9800 6150
-	1    0    0    -1
-$EndComp
-$Comp
-L CONN_1 P8
-U 1 1 513623A1
-P 9800 6250
-F 0 "P8" H 9880 6250 40  0000 L CNN
-F 1 "GPIO1" H 9800 6305 30  0001 C CNN
-F 2 "" H 9800 6250 60  0001 C CNN
-F 3 "" H 9800 6250 60  0001 C CNN
-	1    9800 6250
-	1    0    0    -1
-$EndComp
-$Comp
-L CONN_1 P9
-U 1 1 513623A7
-P 9800 6350
-F 0 "P9" H 9880 6350 40  0000 L CNN
-F 1 "GPIO2" H 9800 6405 30  0001 C CNN
-F 2 "" H 9800 6350 60  0001 C CNN
-F 3 "" H 9800 6350 60  0001 C CNN
-	1    9800 6350
-	1    0    0    -1
-$EndComp
-$Comp
-L CONN_1 P10
-U 1 1 51362518
-P 9800 6450
-F 0 "P10" H 9880 6450 40  0000 L CNN
-F 1 "GPIO3" H 9800 6505 30  0001 C CNN
-F 2 "" H 9800 6450 60  0001 C CNN
-F 3 "" H 9800 6450 60  0001 C CNN
-	1    9800 6450
-	1    0    0    -1
-$EndComp
-Entry Wire Line
-	8950 6250 9050 6150
-Entry Wire Line
-	8950 6350 9050 6250
-Entry Wire Line
-	8950 6450 9050 6350
-Entry Wire Line
-	8950 6550 9050 6450
-Text Label 9150 6150 0    50   ~ 0
-GPIO0
-Text Label 9150 6250 0    50   ~ 0
-GPIO1
-Text Label 9150 6350 0    50   ~ 0
-GPIO2
-Text Label 9150 6450 0    50   ~ 0
-GPIO3
-$Comp
-L CONN_1 P16
-U 1 1 5137B43F
-P 9800 6550
-F 0 "P16" H 9880 6550 40  0000 L CNN
-F 1 "Vcc" H 9800 6605 30  0001 C CNN
-F 2 "" H 9800 6550 60  0001 C CNN
-F 3 "" H 9800 6550 60  0001 C CNN
-	1    9800 6550
-	1    0    0    -1
-$EndComp
-$Comp
-L CONN_1 P17
-U 1 1 5137B445
-P 9800 6650
-F 0 "P17" H 9880 6650 40  0000 L CNN
-F 1 "GND" H 9800 6705 30  0001 C CNN
-F 2 "" H 9800 6650 60  0001 C CNN
-F 3 "" H 9800 6650 60  0001 C CNN
-	1    9800 6650
-	1    0    0    -1
-$EndComp
-$Comp
-L GND #PWR026
-U 1 1 5137B7DB
-P 9300 6850
-F 0 "#PWR026" H 9300 6850 30  0001 C CNN
-F 1 "GND" H 9300 6780 30  0001 C CNN
-F 2 "" H 9300 6850 60  0001 C CNN
-F 3 "" H 9300 6850 60  0001 C CNN
-	1    9300 6850
-	1    0    0    -1
-$EndComp
-$Comp
-L VCC #PWR027
-U 1 1 5137BDF3
-P 8800 6150
-F 0 "#PWR027" H 8800 6250 30  0001 C CNN
-F 1 "VCC" H 8800 6250 30  0000 C CNN
-F 2 "" H 8800 6150 60  0001 C CNN
-F 3 "" H 8800 6150 60  0001 C CNN
-	1    8800 6150
-	1    0    0    -1
-$EndComp
-$Comp
-L VCC #PWR028
+L VCC #PWR026
 U 1 1 516C9166
 P 10850 3050
-F 0 "#PWR028" H 10850 3150 30  0001 C CNN
+F 0 "#PWR026" H 10850 3150 30  0001 C CNN
 F 1 "VCC" H 10850 3150 30  0000 C CNN
 F 2 "" H 10850 3050 60  0001 C CNN
@@
 Wire Bus Line
 	5300 5700 5300 6800
-Wire Wire Line
-	9050 6150 9650 6150
-Wire Wire Line
-	9650 6250 9050 6250
-Wire Wire Line
-	9050 6350 9650 6350
-Wire Wire Line
-	9650 6450 9050 6450
 Wire Bus Line
 	8950 900  8950 6800
 Wire Bus Line
 	8950 6350 8950 6450
-Wire Wire Line
-	9650 6650 9300 6650
-Wire Wire Line
-	9300 6650 9300 6850
-Wire Wire Line
-	9150 6650 9150 6550
-Wire Wire Line
-	9150 6550 9650 6550
-Wire Wire Line
-	8800 6150 8800 6650
-Wire Wire Line
-	8800 6650 9150 6650
 Wire Wire Line
 	9050 3350 9600 3350
@@
 Wire Wire Line
 	9050 1350 9450 1350
-Text Notes 10150 6600 0    60   ~ 0
-Universal expansion\nconnector (bottom)
 Text Notes 9900 1400 0    60   ~ 0
 Backlight expansion\nconnector (top)
@@
 GPIO3
 $Comp
-L VCC #PWR029
+L VCC #PWR027
 U 1 1 51CCBD4D
 P 9350 750
-F 0 "#PWR029" H 9350 850 30  0001 C CNN
+F 0 "#PWR027" H 9350 850 30  0001 C CNN
 F 1 "VCC" H 9350 850 30  0000 C CNN
 F 2 "" H 9350 750 60  0001 C CNN
@@
 	9350 950  9450 950
 $Comp
-L GND #PWR030
+L GND #PWR028
 U 1 1 51CCCE51
 P 9350 1650
-F 0 "#PWR030" H 9350 1650 30  0001 C CNN
+F 0 "#PWR028" H 9350 1650 30  0001 C CNN
 F 1 "GND" H 9350 1580 30  0001 C CNN
 F 2 "" H 9350 1650 60  0001 C CNN
@@
 Connection ~ 10850 5650
 $Comp
-L GND #PWR031
+L GND #PWR029
 U 1 1 523205C7
 P 5650 3050
-F 0 "#PWR031" H 5650 3050 30  0001 C CNN
+F 0 "#PWR029" H 5650 3050 30  0001 C CNN
 F 1 "GND" H 5650 2980 30  0001 C CNN
 F 2 "" H 5650 3050 60  0001 C CNN

Commit message: v0.6
Parts:
- added H1, H2, H3, H4, H5: HOLE, ~, symbol ANYTHING
- added P10: ROW4, symbol CONN_1
- added P11: ROW5, symbol CONN_1
- added P42: GPIO2, symbol CONN_1
- added P43: GPIO3, symbol CONN_1
- added P44: GPIO6, symbol CONN_1
- added P7: ROW1, symbol CONN_1
- added P8: ROW2, symbol CONN_1
- added P9: ROW3, symbol CONN_1
- P18: value Row1 -> LR1
- P19: value Row2 -> LR2
- P20: value Row3 -> LR3
- P21: value Row4 -> LR4
- P23: value Col1 -> LC1
- P24: value Col2 -> LC2
- P25: value Col3 -> LC3
- P26: value Col4 -> LC4
- P27: value Col5 -> LC5
- P28: value Col6 -> LC6
- P29: value Col7 -> LC7
- P30: value Col8 -> LC8
- P31: value Col9 -> LC9
- P32: value Col10 -> LC10
- P33: value Col11 -> LC11
- P34: value Col12 -> LC12
- renumbered P42 to P45
Connections:
- net GND: now also H1.0 (GND), H2.0 (GND), H3.0 (GND), H4.0 (GND), H5.0 (GND)
- net row1: now also P7.1
- net row2: now also P8.1
- net row3: now also P9.1
- net row4: now also P10.1
- net GPIO5: now reaches IC1.22 ((XCK1/~CTS~)PD5)
- net GPIO5: now also P43.1
- net GPIO4: now reaches IC1.26 ((T1/~OC4D~/ADC9)PD6)
- net GPIO4: now also P42.1
- net row5: now reaches IC1.8 ((SS/PCINT0)PB0)
- net row5: now also P11.1
- net MISO renamed GPIO6
- net GPIO6: now also P44.1
- no-connect marks 5 -> 4
Other:
- moved on the sheet: P45

Commit message: v0.7
Parts:
- P42: value GPIO2 -> GPIO4
- P43: value GPIO3 -> GPIO5
- P45: renamed from P11; value ROW5 -> GPIO7
- renumbered P45 to P46
Connections:
- net row5 renamed GPIO7
Other:
- moved on the sheet: P45, P46
Changed lines of the file:
@@
-EESchema Schematic File Version 2  date 10/16/2013 1:34:42 PM
+EESchema Schematic File Version 2  date 10/20/2013 8:52:07 AM
 LIBS:power
 LIBS:mx1a-simple
@@
 encoding utf-8
 Sheet 1 3
-Title "ukbdc - schematic"
-Date "16 oct 2013"
-Rev ""
-Comp "komar"
-Comment1 ""
+Title "The SmallFry 40% Keyboard"
+Date "19 oct 2013"
+Rev "0.7"
+Comp "regack"
+Comment1 "jdcarpe"
 Comment2 ""
 Comment3 ""
@@
 $EndComp
 $Comp
-L CONN_1 P45
+L CONN_1 P46
 U 1 1 51CD1E0B
-P 9600 1750
-F 0 "P45" H 9680 1750 40  0000 L CNN
-F 1 "GND" H 9600 1805 30  0001 C CNN
-F 2 "" H 9600 1750 60  0001 C CNN
-F 3 "" H 9600 1750 60  0001 C CNN
-	1    9600 1750
+P 9600 1900
+F 0 "P46" H 9680 1900 40  0000 L CNN
+F 1 "GND" H 9600 1955 30  0001 C CNN
+F 2 "" H 9600 1900 60  0001 C CNN
+F 3 "" H 9600 1900 60  0001 C CNN
+	1    9600 1900
 	1    0    0    -1
 $EndComp
@@
 Entry Wire Line
 	8950 1350 9050 1250
-Text Notes 9900 1700 0    60   ~ 0
+Text Notes 9900 1850 0    60   ~ 0
 Backlight expansion\nconnector (top)
 Text Label 9100 1050 0    50   ~ 0
@@
 L GND #PWR028
 U 1 1 51CCCE51
-P 9350 1950
-F 0 "#PWR028" H 9350 1950 30  0001 C CNN
-F 1 "GND" H 9350 1880 30  0001 C CNN
-F 2 "" H 9350 1950 60  0001 C CNN
-F 3 "" H 9350 1950 60  0001 C CNN
-	1    9350 1950
+P 9350 2100
+F 0 "#PWR028" H 9350 2100 30  0001 C CNN
+F 1 "GND" H 9350 2030 30  0001 C CNN
+F 2 "" H 9350 2100 60  0001 C CNN
+F 3 "" H 9350 2100 60  0001 C CNN
+	1    9350 2100
 	1    0    0    -1
 $EndComp
@@
 	1    0    0    -1
 $EndComp
-Text Label 6100 4150 2    60   ~ 0
-row5
-Text Label 6650 3450 0    60   ~ 0
-row5
-Entry Wire Line
-	6100 4150 6200 4250
-$Comp
-L CONN_1 P11
+$Comp
+L CONN_1 P45
 U 1 1 525EFFFF
-P 7200 3450
-F 0 "P11" H 7280 3450 40  0000 L CNN
-F 1 "ROW5" H 7200 3505 30  0001 C CNN
-F 2 "" H 7200 3450 60  0001 C CNN
-F 3 "" H 7200 3450 60  0001 C CNN
-	1    7200 3450
-	1    0    0    -1
-$EndComp
-Entry Wire Line
-	6550 3550 6650 3450
+P 9600 1750
+F 0 "P45" H 9680 1750 40  0000 L CNN
+F 1 "GPIO7" H 9600 1805 30  0001 C CNN
+F 2 "" H 9600 1750 60  0001 C CNN
+F 3 "" H 9600 1750 60  0001 C CNN
+	1    9600 1750
+	1    0    0    -1
+$EndComp
 Text Label 5150 4750 2    50   ~ 0
 GPIO4
@@
 P 9600 1450
 F 0 "P42" H 9680 1450 40  0000 L CNN
-F 1 "GPIO2" H 9600 1505 30  0001 C CNN
+F 1 "GPIO4" H 9600 1505 30  0001 C CNN
 F 2 "" H 9600 1450 60  0001 C CNN
 F 3 "" H 9600 1450 60  0001 C CNN
@@
 P 9600 1550
 F 0 "P43" H 9680 1550 40  0000 L CNN
-F 1 "GPIO3" H 9600 1605 30  0001 C CNN
+F 1 "GPIO5" H 9600 1605 30  0001 C CNN
 F 2 "" H 9600 1550 60  0001 C CNN
 F 3 "" H 9600 1550 60  0001 C CNN
@@
 	5200 6150 4750 6150
 Wire Bus Line
-	5300 4700 5300 6800
+	5300 4250 5300 6800
 Wire Bus Line
 	8950 900  8950 6800
@@
 	9350 950  9450 950
 Wire Wire Line
-	9350 1750 9350 1950
-Wire Wire Line
-	9350 1750 9450 1750
+	9350 1900 9350 2100
+Wire Wire Line
+	9350 1900 9450 1900
 Wire Wire Line
 	10850 3050 10850 5850
@@
 	6650 3050 7050 3050
 Wire Wire Line
-	6100 4150 5400 4150
-Wire Wire Line
-	5400 4150 5400 4250
-Wire Wire Line
-	5400 4250 5200 4250
-Wire Wire Line
-	5200 4250 5200 4150
-Wire Wire Line
-	5200 4150 4750 4150
-Wire Wire Line
-	7050 3450 6650 3450
-Wire Wire Line
 	5200 4750 4750 4750
 Wire Wire Line
@@
 Wire Wire Line
 	6700 3550 6650 3550
+Wire Wire Line
+	4750 4150 4850 4150
+Wire Wire Line
+	4850 4150 4850 4200
+Wire Wire Line
+	4850 4200 5200 4200
+Entry Wire Line
+	5200 4200 5300 4300
+Text Label 9100 1750 0    50   ~ 0
+GPIO7
+Wire Wire Line
+	9050 1750 9450 1750
+Entry Wire Line
+	8950 1850 9050 1750
+Text Label 5200 4200 2    50   ~ 0
+GPIO7
 $EndSCHEMATC

Commit message: v0.10
Parts:
- removed P204, P205: GND, symbol CONN_1
- added P35: LGND, symbol CONN_1
- added P36: LVcc, symbol CONN_1
- added P46: GPIO8(SDA), symbol CONN_1
- P42: value GPIO4 -> GPIO4(SS)
- P43: value GPIO5 -> GPIO5(SCK)
- P44: value GPIO6 -> GPIO6(MOSI)
- P45: value GPIO7 -> GPIO7(SCL)
- renumbered P46 to P47
Connections:
- net MOSI is gone; now on net GPIO6: IC1.10 ((PDI/PCINT2/MOSI)PB2), P4.1
- net SCK is gone; now on net GPIO5: IC1.9 ((PCINT1/SCLK)PB1), P3.1
- net col12 is gone; now on net GPIO1: IC1.27 ((T0/OC4D/ADC10)PD7)
- net col7 is gone; now on net row3: IC1.25 ((ICP1/ADC8)PD4)
- net GND: now also P35.1
- net GPIO0: now also IC1.26 ((T1/~OC4D~/ADC9)PD6); no longer IC1.36 ((ADC7/TDI)PF7)
- net GPIO1: no longer IC1.37 ((ADC6/TDO)PF6)
- net GPIO2: now also IC1.1 ((INT6/AIN0)PE6); no longer IC1.38 ((ADC5/TMS)PF5)
- net GPIO3: now also IC1.32 ((ICP3/CLK0/OC4A)PC7); no longer IC1.39 ((ADC4/TCK)PF4)
- net GPIO4: now also IC1.8 ((SS/PCINT0)PB0); no longer IC1.26 ((T1/~OC4D~/ADC9)PD6)
- net GPIO5: no longer IC1.22 ((XCK1/~CTS~)PD5)
- net GPIO6: no longer IC1.11 ((PDO/PCINT3/MISO)PB3), P1.1
- net GPIO7: now also IC1.18 ((OC0B/SCL/INT0)PD0); no longer IC1.8 ((SS/PCINT0)PB0)
- net VCC: now also P36.1
- net col10: now also IC1.30 ((PCINT6/OC1B/OC4B/ADC13)PB6); no longer IC1.29 ((PCINT5/OC1A/~OC4B~/ADC12)PB5)
- net col11: now also IC1.12 ((PCINT7/OC0A/OC1C/~RTS~)PB7); no longer IC1.28 ((PCINT4/ADC11)PB4)
- net col3: now also IC1.39 ((ADC4/TCK)PF4); no longer IC1.1 ((INT6/AIN0)PE6)
- net col4: now also IC1.38 ((ADC5/TMS)PF5); no longer IC1.32 ((ICP3/CLK0/OC4A)PC7)
- net col5: now also IC1.37 ((ADC6/TDO)PF6); no longer IC1.31 ((OC3A/~OC4A~)PC6)
- net col6: now also IC1.36 ((ADC7/TDI)PF7); no longer IC1.30 ((PCINT6/OC1B/OC4B/ADC13)PB6)
- net col9: now also IC1.29 ((PCINT5/OC1A/~OC4B~/ADC12)PB5); no longer IC1.12 ((PCINT7/OC0A/OC1C/~RTS~)PB7)
- net row1: now also IC1.20 ((RXD1/INT2)PD2); no longer IC1.18 ((OC0B/SCL/INT0)PD0)
- net row2: now also IC1.21 ((TXD1/INT3)PD3); no longer IC1.19 ((SDA/INT1)PD1)
- net row3: no longer IC1.20 ((RXD1/INT2)PD2)
- net row4: now also IC1.22 ((XCK1/~CTS~)PD5); no longer IC1.21 ((TXD1/INT3)PD3)
- new net GPIO8: IC1.19 ((SDA/INT1)PD1), P46.1
- new net MISO: IC1.11 ((PDO/PCINT3/MISO)PB3), P1.1
- new net caps: IC1.31 ((OC3A/~OC4A~)PC6)
- new net col8: IC1.28 ((PCINT4/ADC11)PB4)
Other:
- note added: "Expansion\nconnector \n(right)"
- note added: "Ground Pins"
- note added: "ISP Pins"
- note added: "LED Matrix\n(top)"
- note added: "Mounting\nHoles"
- note added: "PWM"
- note added: "SW01 LED (ESCAPE)\n"
- note added: "WASD Cluster LEDs\n"
- note removed: "Backlight expansion\nconnector (top)"
- moved on the sheet: H1, H2, H3, H4, H5, P47, R3
