File: matrix.sch (KiCad schematic (older format))
At the start: 82 parts

Commit message: v0.4
Parts:
- added S481, S531: MX1A, symbol MX1A
Connections:
- net col10: now also D48.2 (K); no longer D48.1 (A)
- net col11: now also D53.2 (K); no longer D53.1 (A)
- net row3: now also S481.1, S531.1
- net at S48.2: now also D48.1 (A), S481.2; no longer D48.2 (K)
- net at S53.2: now also D53.1 (A), S531.2; no longer D53.2 (K)
Other:
- moved on the sheet: D48, D53
Changed lines of the file:
@@
-EESchema Schematic File Version 2  date 9/13/2013 12:58:58 PM
+EESchema Schematic File Version 2  date 9/20/2013 9:26:54 AM
 LIBS:power
 LIBS:mx1a-simple
@@
 Sheet 2 3
 Title ""
-Date "13 sep 2013"
+Date "20 sep 2013"
 Rev ""
 Comp ""
@@
 L DIODE D48
 U 1 1 506B59AA
-P 9650 5550
-F 0 "D48" H 9500 5500 40  0000 C CNN
-F 1 "1N4148" H 9550 5550 40  0000 C CNN
-F 2 "" H 9650 5550 60  0001 C CNN
-F 3 "" H 9650 5550 60  0001 C CNN
-F 4 "DC Components" H 4700 4350 60  0001 C CNN "Vendor"
-F 5 "CD4148WS(0805C)" H 4700 4350 60  0001 C CNN "Product"
-F 6 "TME" H 4700 4350 60  0001 C CNN "Supplier"
-F 7 "1N4148-0805" H 4700 4350 60  0001 C CNN "Supplier Symbol"
-	1    9650 5550
+P 9650 6000
+F 0 "D48" H 9500 5950 40  0000 C CNN
+F 1 "1N4148" H 9550 6000 40  0000 C CNN
+F 2 "" H 9650 6000 60  0001 C CNN
+F 3 "" H 9650 6000 60  0001 C CNN
+F 4 "DC Components" H 4700 4800 60  0001 C CNN "Vendor"
+F 5 "CD4148WS(0805C)" H 4700 4800 60  0001 C CNN "Product"
+F 6 "TME" H 4700 4800 60  0001 C CNN "Supplier"
+F 7 "1N4148-0805" H 4700 4800 60  0001 C CNN "Supplier Symbol"
+	1    9650 6000
 	1    0    0    -1
 $EndComp
@@
 L DIODE D53
 U 1 1 506B5A31
-P 10350 5550
-F 0 "D53" H 10200 5500 40  0000 C CNN
-F 1 "1N4148" H 10250 5550 40  0000 C CNN
-F 2 "" H 10350 5550 60  0001 C CNN
-F 3 "" H 10350 5550 60  0001 C CNN
-F 4 "DC Components" H 4850 4350 60  0001 C CNN "Vendor"
-F 5 "CD4148WS(0805C)" H 4850 4350 60  0001 C CNN "Product"
-F 6 "TME" H 4850 4350 60  0001 C CNN "Supplier"
-F 7 "1N4148-0805" H 4850 4350 60  0001 C CNN "Supplier Symbol"
-	1    10350 5550
+P 10350 6000
+F 0 "D53" H 10200 5950 40  0000 C CNN
+F 1 "1N4148" H 10250 6000 40  0000 C CNN
+F 2 "" H 10350 6000 60  0001 C CNN
+F 3 "" H 10350 6000 60  0001 C CNN
+F 4 "DC Components" H 4850 4800 60  0001 C CNN "Vendor"
+F 5 "CD4148WS(0805C)" H 4850 4800 60  0001 C CNN "Product"
+F 6 "TME" H 4850 4800 60  0001 C CNN "Supplier"
+F 7 "1N4148-0805" H 4850 4800 60  0001 C CNN "Supplier Symbol"
+	1    10350 6000
 	1    0    0    -1
 $EndComp
@@
 	10550 4550 10550 4400
 Wire Wire Line
-	9450 5550 9450 5650
-Wire Wire Line
-	9450 5650 9900 5650
-Wire Wire Line
-	9850 5550 9850 5400
+	9850 5400 9850 5900
 Wire Wire Line
 	8750 7050 8750 7150
@@
 	9850 7050 9850 6900
 Wire Wire Line
-	10150 5550 10150 5650
-Wire Wire Line
-	10150 5650 10600 5650
-Wire Wire Line
-	10550 5550 10550 5400
+	10550 5400 10550 5900
 Wire Wire Line
 	10850 3350 10850 3450
@@
 Connection ~ 9200 4650
 Connection ~ 9200 5650
-Connection ~ 9900 5650
-Connection ~ 10600 5650
 Connection ~ 10600 7150
 Connection ~ 9900 7150
@@
 Wire Wire Line
 	3600 7150 3600 1400
+$Comp
+L MX1A S531
+U 1 1 523C5315
+P 10350 5850
+F 0 "S531" H 10200 6100 60  0000 C CNN
+F 1 "MX1A" H 10350 5950 60  0000 C CNN
+F 2 "" H 10350 5850 60  0001 C CNN
+F 3 "" H 10350 5850 60  0001 C CNN
+	1    10350 5850
+	1    0    0    -1
+$EndComp
+$Comp
+L MX1A S481
+U 1 1 523C531B
+P 9650 5850
+F 0 "S481" H 9500 6100 60  0000 C CNN
+F 1 "MX1A" H 9650 5950 60  0000 C CNN
+F 2 "" H 9650 5850 60  0001 C CNN
+F 3 "" H 9650 5850 60  0001 C CNN
+	1    9650 5850
+	1    0    0    -1
+$EndComp
+Wire Wire Line
+	10150 5450 10100 5450
+Wire Wire Line
+	10100 5450 10100 5150
+Connection ~ 10100 5150
+Wire Wire Line
+	9400 5150 9400 5450
+Wire Wire Line
+	9400 5450 9450 5450
+Connection ~ 9400 5150
+Wire Wire Line
+	9850 5900 9450 5900
+Wire Wire Line
+	9450 5900 9450 6000
+Connection ~ 9850 5700
+Wire Wire Line
+	9850 6000 9900 6000
+Connection ~ 9900 6000
+Wire Wire Line
+	10150 6000 10150 5900
+Wire Wire Line
+	10150 5900 10550 5900
+Connection ~ 10550 5700
+Wire Wire Line
+	10550 6000 10600 6000
+Connection ~ 10600 6000
 $EndSCHEMATC

Commit message: v0.10
Connections:
- net col12 is gone; now on net col11: D56.1 (A)
- net row1: no longer S56.1
- net row4: now also S56.1
Other:
- note added: "S03 (CAPS) LED\n"
- moved on the sheet: D56, S56
Changed lines of the file:
@@
-EESchema Schematic File Version 2  date 10/20/2013 8:52:07 AM
+EESchema Schematic File Version 2  date 11/23/2013 1:19:47 PM
 LIBS:power
 LIBS:mx1a-simple
@@
 LIBS:atmega32u4
 LIBS:dtsjw
-LIBS:oupiin_usb
 LIBS:device
 LIBS:conn
@@
 Sheet 2 3
 Title "The SmallFry 40% Keyboard"
-Date "19 oct 2013"
-Rev "0.7"
+Date "23 nov 2013"
+Rev "0.10"
 Comp "regack"
 Comment1 "jdcarpe"
@@
 L MX1A S56
 U 1 1 5040DDD9
-P 11050 3350
-F 0 "S56" H 10900 3600 60  0000 C CNN
-F 1 "MX1A" H 11050 3450 60  0000 C CNN
-F 2 "" H 11050 3350 60  0001 C CNN
-F 3 "" H 11050 3350 60  0001 C CNN
-	1    11050 3350
+P 10350 7050
+F 0 "S56" H 10200 7300 60  0000 C CNN
+F 1 "MX1A" H 10350 7150 60  0000 C CNN
+F 2 "" H 10350 7050 60  0001 C CNN
+F 3 "" H 10350 7050 60  0001 C CNN
+	1    10350 7050
 	1    0    0    -1
 $EndComp
@@
 Text HLabel 10600 1400 1    60   3State ~ 0
 col11
-Text HLabel 11300 1400 1    60   3State ~ 0
-col12
-$Comp
-L VCC #PWR030
+$Comp
+L VCC #PWR032
 U 1 1 5043970C
 P 12550 3550
-F 0 "#PWR030" H 12550 3650 30  0001 C CNN
+F 0 "#PWR032" H 12550 3650 30  0001 C CNN
 F 1 "VCC" H 12550 3650 30  0000 C CNN
 F 2 "" H 12550 3550 60  0001 C CNN
@@
 L DIODE D56
 U 1 1 506B5A67
-P 11050 3350
-F 0 "D56" H 10900 3300 40  0000 C CNN
-F 1 "1N4148" H 10950 3350 40  0000 C CNN
-F 2 "" H 11050 3350 60  0001 C CNN
-F 3 "" H 11050 3350 60  0001 C CNN
-F 4 "DC Components" H 5000 3350 60  0001 C CNN "Vendor"
-F 5 "CD4148WS(0805C)" H 5000 3350 60  0001 C CNN "Product"
-F 6 "TME" H 5000 3350 60  0001 C CNN "Supplier"
-F 7 "1N4148-0805" H 5000 3350 60  0001 C CNN "Supplier Symbol"
-	1    11050 3350
+P 10350 7050
+F 0 "D56" H 10200 7000 40  0000 C CNN
+F 1 "1N4148" H 10250 7050 40  0000 C CNN
+F 2 "" H 10350 7050 60  0001 C CNN
+F 3 "" H 10350 7050 60  0001 C CNN
+F 4 "DC Components" H 4300 7050 60  0001 C CNN "Vendor"
+F 5 "CD4148WS(0805C)" H 4300 7050 60  0001 C CNN "Product"
+F 6 "TME" H 4300 7050 60  0001 C CNN "Supplier"
+F 7 "1N4148-0805" H 4300 7050 60  0001 C CNN "Supplier Symbol"
+	1    10350 7050
 	1    0    0    -1
 $EndComp
@@
 Text Notes 10200 3700 0    60   ~ 0
 P
-Text Notes 10850 3700 0    60   ~ 0
+Text Notes 10750 3250 0    60   ~ 0
 BKSP
 Text Notes 3200 5900 0    60   ~ 0
@@
 	10550 5400 10550 5900
 Wire Wire Line
-	10850 3350 10850 3450
-Wire Wire Line
-	10850 3450 11300 3450
-Wire Wire Line
-	11250 3350 11250 3200
+	10150 7050 10150 7150
+Wire Wire Line
+	10150 7150 10600 7150
+Wire Wire Line
+	10550 7050 10550 6900
 Connection ~ 3600 3450
 Connection ~ 4300 3450
@@
 	10550 6000 10600 6000
 Connection ~ 10600 6000
+Text Notes 10250 7400 0    60   ~ 0
+BKSP
+Wire Notes Line
+	10500 7350 11600 7350
+Wire Notes Line
+	11600 7350 11600 3200
+Wire Notes Line
+	11600 3200 11000 3200
+Connection ~ 10150 6650
+Text Notes 12750 4250 0    120  ~ 0
+S03 (CAPS) LED\n
 $EndSCHEMATC
